File: main/main.sch (KiCad schematic (older format))
At the start: 14 parts, among them J1 PROG, SW1 CONFIG, U1 MSP430FR2311IPW16R, U2 RFM64W

Commit message: Replaced github libs for local ones and assigned footprints
Parts:
- ANT1: footprint Housings_SSOP:TSSOP-16_4.4x5mm_Pitch0.65mm -> Connector_Wire:SolderWirePad_1x01_Drill0.8mm
- BT1: footprint (none) -> Connector_Wire:SolderWirePad_1x02_P5.08mm_Drill1.5mm
- J1: footprint (none) -> Connector_PinHeader_2.54mm:PinHeader_1x04_P2.54mm_Vertical
- SW1: footprint (none) -> Button_Switch_SMD:SW_SPST_EVPBF
- U1: footprint (none) -> Package_SO:TSSOP-16_4.4x5mm_P0.65mm
- U2: footprint (none) -> Custom_RF:RFM64W-433S2
Changed lines of the file:
@@
 F 0 "U2" H 2050 3500 50  0000 C CNN
 F 1 "RFM64W" H 2050 2300 50  0000 C CNN
-F 2 "" H 2050 2950 50  0001 C CNN
+F 2 "Custom_RF:RFM64W-433S2" H 2050 2950 50  0001 C CNN
 F 3 "" H 2050 2950 50  0001 C CNN
 	1    2050 2950
@@
 F 0 "ANT1" H 2900 2250 50  0000 L CNN
 F 1 "433MHz_HELICOIDAL" H 2850 2450 50  0000 C CNN
-F 2 "Housings_SSOP:TSSOP-16_4.4x5mm_Pitch0.65mm" H 2850 2300 50  0001 C CNN
+F 2 "Connector_Wire:SolderWirePad_1x01_Drill0.8mm" H 2850 2300 50  0001 C CNN
 F 3 "~" H 2850 2300 50  0001 C CNN
 	1    2850 2300
@@
 F 0 "U1" H 1900 2550 60  0000 C CNN
 F 1 "MSP430FR2311IPW16R" H 1850 1650 60  0000 C CNN
-F 2 "" H 1400 1700 60  0001 C CNN
+F 2 "Package_SO:TSSOP-16_4.4x5mm_P0.65mm" H 1400 1700 60  0001 C CNN
 F 3 "" H 1400 1700 60  0001 C CNN
 	1    1900 1700
@@
 F 0 "SW1" H 5550 3450 50  0000 C CNN
 F 1 "CONFIG" H 5550 3750 50  0000 C CNN
-F 2 "" H 5550 3750 50  0001 C CNN
+F 2 "Button_Switch_SMD:SW_SPST_EVPBF" H 5550 3750 50  0001 C CNN
 F 3 "" H 5550 3750 50  0001 C CNN
 	1    5550 3550
@@
 F 0 "BT1" H 4700 3800 50  0000 L CNN
 F 1 "CR2477" V 4450 3700 50  0000 C CNN
-F 2 "" V 4600 3710 50  0001 C CNN
+F 2 "Connector_Wire:SolderWirePad_1x02_P5.08mm_Drill1.5mm" V 4600 3710 50  0001 C CNN
 F 3 "~" V 4600 3710 50  0001 C CNN
 	1    4600 3650
@@
 F 0 "J1" H 4600 2500 50  0000 C CNN
 F 1 "PROG" V 4700 2250 50  0000 C CNN
-F 2 "" H 4600 2300 50  0001 C CNN
+F 2 "Connector_PinHeader_2.54mm:PinHeader_1x04_P2.54mm_Vertical" H 4600 2300 50  0001 C CNN
 F 3 "~" H 4600 2300 50  0001 C CNN
 	1    4600 2300

Commit message: Added board layout
Parts:
- removed C3: 10u, Capacitors_SMD:C_0805_HandSoldering, symbol Device:C
- C1, C2: footprint Capacitors_SMD:C_0805_HandSoldering -> Capacitor_SMD:C_0805_2012Metric
- D1: footprint LEDs:LED_0805_HandSoldering -> LED_SMD:LED_0805_2012Metric
- D2: footprint LEDs:LED_D3.0mm -> LED_THT:LED_D3.0mm
- R1, R2, R3: footprint Resistors_SMD:R_0805_HandSoldering -> Resistor_SMD:R_0805_2012Metric
Connections:
- wire segments 69 -> 67
Changed lines of the file:
@@
 L Device:LED D2
 U 1 1 5AEB1646
-P 5500 1550
-F 0 "D2" V 5538 1432 50  0000 R CNN
-F 1 "IR" V 5447 1432 50  0000 R CNN
-F 2 "LEDs:LED_D3.0mm" H 5500 1550 50  0001 C CNN
-F 3 "~" H 5500 1550 50  0001 C CNN
-	1    5500 1550
+P 5500 1050
+F 0 "D2" V 5538 932 50  0000 R CNN
+F 1 "IR" V 5447 932 50  0000 R CNN
+F 2 "LED_THT:LED_D3.0mm" H 5500 1050 50  0001 C CNN
+F 3 "~" H 5500 1050 50  0001 C CNN
+	1    5500 1050
 	0    -1   -1   0
 $EndComp
@@
 L Device:LED D1
 U 1 1 5AEB16CA
-P 4450 1550
-F 0 "D1" V 4488 1432 50  0000 R CNN
-F 1 "RED" V 4397 1432 50  0000 R CNN
-F 2 "LEDs:LED_0805_HandSoldering" H 4450 1550 50  0001 C CNN
-F 3 "~" H 4450 1550 50  0001 C CNN
-	1    4450 1550
+P 4500 1050
+F 0 "D1" V 4538 932 50  0000 R CNN
+F 1 "RED" V 4447 932 50  0000 R CNN
+F 2 "LED_SMD:LED_0805_2012Metric" H 4500 1050 50  0001 C CNN
+F 3 "~" H 4500 1050 50  0001 C CNN
+	1    4500 1050
 	0    -1   -1   0
 $EndComp
@@
 $EndComp
 $Comp
-L Device:C C3
-U 1 1 5AEB1EB0
-P 3550 2500
-F 0 "C3" H 3600 2600 50  0000 L CNN
-F 1 "10u" H 3600 2400 50  0000 L CNN
-F 2 "Capacitors_SMD:C_0805_HandSoldering" H 3588 2350 50  0001 C CNN
-F 3 "~" H 3550 2500 50  0001 C CNN
-	1    3550 2500
-	1    0    0    -1
-$EndComp
-$Comp
-L power:GND #PWR014
-U 1 1 5AEB200B
-P 3550 2700
-F 0 "#PWR014" H 3550 2450 50  0001 C CNN
-F 1 "GND" H 3555 2527 50  0000 C CNN
-F 2 "" H 3550 2700 50  0001 C CNN
-F 3 "" H 3550 2700 50  0001 C CNN
-	1    3550 2700
-	1    0    0    -1
-$EndComp
-Wire Wire Line
-	3550 2300 3550 2350
-Wire Wire Line
-	3550 2700 3550 2650
-$Comp
 L Device:Battery_Cell BT1
 U 1 1 5AEB2D3B
@@
 $EndComp
 $Comp
-L power:VDD #PWR013
-U 1 1 5AEB489D
-P 3550 2300
-F 0 "#PWR013" H 3550 2150 50  0001 C CNN
-F 1 "VDD" H 3550 2450 50  0000 C CNN
-F 2 "" H 3550 2300 50  0001 C CNN
-F 3 "" H 3550 2300 50  0001 C CNN
-	1    3550 2300
-	1    0    0    -1
-$EndComp
-$Comp
 L power:VDD #PWR011
 U 1 1 5AEB4A6F
@@
 Wire Wire Line
 	5550 3800 5550 3750
-Wire Wire Line
-	5500 1750 5500 1700
 Wire Notes Line
 	4000 3050 4950 3050
@@
 BATTERY
 Wire Notes Line
-	3400 2050 3400 2950
-Wire Notes Line
 	750  3750 750  2050
 Text Notes 750  2050 0    50   ~ 0
@@
 Wire Notes Line
 	750  3750 3800 3750
-Wire Notes Line
-	3800 2950 3400 2950
 Wire Notes Line
 	750  750  3800 750
@@
 F 0 "C1" H 3250 1300 50  0000 L CNN
 F 1 "10u" H 3250 1100 50  0000 L CNN
-F 2 "Capacitors_SMD:C_0805_HandSoldering" H 3238 1050 50  0001 C CNN
+F 2 "Capacitor_SMD:C_0805_2012Metric" H 3238 1050 50  0001 C CNN
 F 3 "~" H 3200 1200 50  0001 C CNN
 	1    3200 1200
@@
 F 0 "C2" H 3550 1300 50  0000 L CNN
 F 1 "100n" H 3550 1100 50  0000 L CNN
-F 2 "Capacitors_SMD:C_0805_HandSoldering" H 3538 1050 50  0001 C CNN
+F 2 "Capacitor_SMD:C_0805_2012Metric" H 3538 1050 50  0001 C CNN
 F 3 "~" H 3500 1200 50  0001 C CNN
 	1    3500 1200
@@
 SCLK
 Text Label 900  1650 0    50   ~ 0
-NSS_CFG
+IRQ_1
 Text Label 900  1550 0    50   ~ 0
-POR
+IRQ_0
 Text Label 2900 1150 2    50   ~ 0
-IRQ_0
+IR
 Text Label 2900 1050 2    50   ~ 0
-IRQ_1
+STATUS
 NoConn ~ 2900 1350
 Text Label 900  1450 0    50   ~ 0
@@
 TST
 Text Label 900  950  0    50   ~ 0
-PB_CFG
+NSS_CFG
 Text Label 900  1050 0    50   ~ 0
-STATUS
+POR
 Wire Wire Line
 	5550 3300 5200 3300
@@
 L Device:R R2
 U 1 1 5AEE3CE2
-P 5500 1200
-F 0 "R2" H 5570 1246 50  0000 L CNN
-F 1 "1k" H 5570 1155 50  0000 L CNN
-F 2 "Resistors_SMD:R_0805_HandSoldering" V 5430 1200 50  0001 C CNN
-F 3 "~" H 5500 1200 50  0001 C CNN
-	1    5500 1200
-	1    0    0    -1
-$EndComp
-Wire Wire Line
-	5500 1350 5500 1400
+P 5500 1400
+F 0 "R2" H 5570 1446 50  0000 L CNN
+F 1 "1k" H 5570 1355 50  0000 L CNN
+F 2 "Resistor_SMD:R_0805_2012Metric" V 5430 1400 50  0001 C CNN
+F 3 "~" H 5500 1400 50  0001 C CNN
+	1    5500 1400
+	1    0    0    -1
+$EndComp
 $Comp
 L Device:R R1
 U 1 1 5AEE464D
-P 4450 1200
-F 0 "R1" H 4520 1246 50  0000 L CNN
-F 1 "1k" H 4520 1155 50  0000 L CNN
-F 2 "Resistors_SMD:R_0805_HandSoldering" V 4380 1200 50  0001 C CNN
-F 3 "~" H 4450 1200 50  0001 C CNN
-	1    4450 1200
-	1    0    0    -1
-$EndComp
-Wire Wire Line
-	4450 1350 4450 1400
-Wire Wire Line
-	4450 1700 4450 1750
-Wire Wire Line
-	4450 1750 4050 1750
-Text Label 4050 1750 0    50   ~ 0
+P 4500 1400
+F 0 "R1" H 4570 1446 50  0000 L CNN
+F 1 "1k" H 4570 1355 50  0000 L CNN
+F 2 "Resistor_SMD:R_0805_2012Metric" V 4430 1400 50  0001 C CNN
+F 3 "~" H 4500 1400 50  0001 C CNN
+	1    4500 1400
+	1    0    0    -1
+$EndComp
+Text Label 4100 850  0    50   ~ 0
 STATUS
-$Comp
-L power:VDD #PWR04
-U 1 1 5AEE72F9
-P 4450 1000
-F 0 "#PWR04" H 4450 850 50  0001 C CNN
-F 1 "VDD" H 4450 1150 50  0000 C CNN
-F 2 "" H 4450 1000 50  0001 C CNN
-F 3 "" H 4450 1000 50  0001 C CNN
-	1    4450 1000
-	1    0    0    -1
-$EndComp
-Wire Wire Line
-	4450 1000 4450 1050
 Wire Wire Line
 	4400 2200 4200 2200
@@
 	4400 2300 4200 2300
 Text Label 4200 2300 0    50   ~ 0
-TST
+RST
 Wire Wire Line
 	4400 2400 4200 2400
 Text Label 4200 2400 0    50   ~ 0
-RST
+TST
 Wire Wire Line
 	4400 2500 4200 2500
@@
 F 0 "R3" H 5670 2546 50  0000 L CNN
 F 1 "100k" H 5670 2455 50  0000 L CNN
-F 2 "Resistors_SMD:R_0805_HandSoldering" V 5530 2500 50  0001 C CNN
+F 2 "Resistor_SMD:R_0805_2012Metric" V 5530 2500 50  0001 C CNN
 F 3 "~" H 5600 2500 50  0001 C CNN
 	1    5600 2500
@@
 Text Notes 4000 750  0    50   ~ 0
 STATUS LED
-$Comp
-L power:VDD #PWR0102
-U 1 1 5AFCAF1B
-P 5500 1000
-F 0 "#PWR0102" H 5500 850 50  0001 C CNN
-F 1 "VDD" H 5517 1173 50  0000 C CNN
-F 2 "" H 5500 1000 50  0001 C CNN
-F 3 "" H 5500 1000 50  0001 C CNN
-	1    5500 1000
-	1    0    0    -1
-$EndComp
-Wire Wire Line
-	5500 1000 5500 1050
 Wire Notes Line
 	5050 750  5050 1850
@@
 Wire Notes Line
 	6000 750  5050 750
-Wire Wire Line
-	5500 1750 5100 1750
-Text Label 5100 1750 0    50   ~ 0
+Text Label 5150 850  0    50   ~ 0
 IR
 Text Label 2900 950  2    50   ~ 0
-IR
+PB_CFG
 Text Notes 5050 750  0    50   ~ 0
 INFRA-RED LED
+$Comp
+L power:GND #PWR0102
+U 1 1 5AFAF5A6
+P 4500 1600
+F 0 "#PWR0102" H 4500 1350 50  0001 C CNN
+F 1 "GND" H 4500 1450 50  0000 C CNN
+F 2 "" H 4500 1600 50  0001 C CNN
+F 3 "" H 4500 1600 50  0001 C CNN
+	1    4500 1600
+	1    0    0    -1
+$EndComp
+Wire Wire Line
+	4500 850  4500 900
+Wire Wire Line
+	4100 850  4500 850
+Wire Wire Line
+	4500 1200 4500 1250
+Wire Wire Line
+	4500 1600 4500 1550
+Wire Wire Line
+	5500 900  5500 850
+Wire Wire Line
+	5500 850  5150 850
+Wire Wire Line
+	5500 1250 5500 1200
+$Comp
+L power:GND #PWR0103
+U 1 1 5AFBA3CA
+P 5500 1600
+F 0 "#PWR0103" H 5500 1350 50  0001 C CNN
+F 1 "GND" H 5500 1450 50  0000 C CNN
+F 2 "" H 5500 1600 50  0001 C CNN
+F 3 "" H 5500 1600 50  0001 C CNN
+	1    5500 1600
+	1    0    0    -1
+$EndComp
+Wire Wire Line
+	5500 1600 5500 1550
 $EndSCHEMATC

Commit message: Updated footprints in schematic
Parts:
- BT1: footprint Connector_Wire:SolderWirePad_1x02_P5.08mm_Drill1.5mm -> Connector_PinHeader_2.00mm:PinHeader_1x02_P2.00mm_Vertical
- J1: footprint Connector_PinHeader_2.54mm:PinHeader_1x04_P2.54mm_Vertical -> Connector_PinHeader_1.27mm:PinHeader_1x04_P1.27mm_Vertical
Changed lines of the file:
@@
 F 0 "BT1" H 4700 3800 50  0000 L CNN
 F 1 "CR2477" V 4450 3700 50  0000 C CNN
-F 2 "Connector_Wire:SolderWirePad_1x02_P5.08mm_Drill1.5mm" V 4600 3710 50  0001 C CNN
+F 2 "Connector_PinHeader_2.00mm:PinHeader_1x02_P2.00mm_Vertical" V 4600 3710 50  0001 C CNN
 F 3 "~" V 4600 3710 50  0001 C CNN
 	1    4600 3650
@@
 F 0 "J1" H 4600 2500 50  0000 C CNN
 F 1 "PROG" V 4700 2250 50  0000 C CNN
-F 2 "Connector_PinHeader_2.54mm:PinHeader_1x04_P2.54mm_Vertical" H 4600 2300 50  0001 C CNN
+F 2 "Connector_PinHeader_1.27mm:PinHeader_1x04_P1.27mm_Vertical" H 4600 2300 50  0001 C CNN
 F 3 "~" H 4600 2300 50  0001 C CNN
 	1    4600 2300

Commit message: Handmade version of RF BoosterPack for MSP-EXP430FR2311 board
Parts:
- removed J1: PROG, Connector_PinHeader_1.27mm:PinHeader_1x04_P1.27mm_Vertical, symbol Connector_Generic:Conn_01x04
- removed U1: MSP430FR2311IPW16R, Package_SO:TSSOP-16_4.4x5mm_P0.65mm, symbol Custom_Microcontroller:MSP430FR2311IPW16R
- added R4, R5, R6, R7, R8: 0, Resistor_SMD:R_1206_3216Metric_Pad1.24x1.80mm_HandSolder, symbol Device:R
- added U1: MSP-EXP430FR2311_BoosterPack, Custom_BoosterPack:BoosterPack_20pins, symbol Custom_MSP-EXP430FR2311_BoosterPack:MSP-EXP430FR2311_BoosterPack
- ANT1: footprint Connector_Wire:SolderWirePad_1x01_Drill0.8mm -> Connector_Wire:SolderWirePad_single_0-8mmDrill
- BT1: footprint Connector_PinHeader_2.00mm:PinHeader_1x02_P2.00mm_Vertical -> Connector_PinHeader_2.54mm:PinHeader_1x02_P2.54mm_Vertical
- C1: footprint Capacitor_SMD:C_0805_2012Metric -> Capacitor_THT:CP_Radial_D4.0mm_P2.00mm
- C2: footprint Capacitor_SMD:C_0805_2012Metric -> Capacitor_SMD:C_0805_2012Metric_Pad1.15x1.50mm_HandSolder
- D1: footprint LED_SMD:LED_0805_2012Metric -> LED_THT:LED_D5.0mm
- D2: footprint LED_THT:LED_D3.0mm -> LED_THT:LED_D5.0mm
- R1, R2, R3: footprint Resistor_SMD:R_0805_2012Metric -> Resistor_SMD:R_0805_2012Metric_Pad1.15x1.50mm_HandSolder
Connections:
- net labels removed: RST, TST
- no-connect marks 3 -> 8
Other:
- note added: "R: 0805\nC 10u: eletrolitico 4mm (medir)\nSW: 6x6mm smd (duqueeletronica)\nLEDs: 5mm\nBAT: deixar conectores"
- note removed: "PROG. HEADER"

Commit message: Updated BoosterPack board layout
Parts:
- removed R4, R5, R6, R7, R8: 0, Resistor_SMD:R_1206_3216Metric_Pad1.24x1.80mm_HandSolder, symbol Device:R
- SW1: footprint Button_Switch_SMD:SW_SPST_EVPBF -> Custom_SwitchButton:SwitchButton_SMD_4x4mm
Connections:
- wire segments 67 -> 66
Other:
- note removed: "R: 0805\nC 10u: eletrolitico 4mm (medir)\nSW: 6x6mm smd (duqueeletronica)\nLEDs: 5mm\nBAT: deixar conectores"
Changed lines of the file:
@@
 F 0 "SW1" H 4500 4150 50  0000 C CNN
 F 1 "CONFIG" H 4500 4450 50  0000 C CNN
-F 2 "Button_Switch_SMD:SW_SPST_EVPBF" H 4500 4450 50  0001 C CNN
+F 2 "Custom_SwitchButton:SwitchButton_SMD_4x4mm" H 4500 4450 50  0001 C CNN
 F 3 "" H 4500 4450 50  0001 C CNN
 	1    4500 4250
@@
 	1    0    0    -1
 $EndComp
-Wire Wire Line
-	4500 3750 4500 3700
 $Comp
 L power:GND #PWR03
@@
 $EndComp
 Wire Wire Line
-	4500 850  4500 900
-Wire Wire Line
 	4100 850  4500 850
 Wire Wire Line
@@
 	1    0    0    -1
 $EndComp
-Text Label 2650 1850 2    50   ~ 0
+Text Label 2650 1750 2    50   ~ 0
 NSS_CFG
-Text Label 900  1350 0    50   ~ 0
-POR
+Text Label 2650 1150 2    50   ~ 0
+IR
 Text Label 900  950  0    50   ~ 0
 VDD
 Text Label 2650 950  2    50   ~ 0
 GND
+Text Label 2650 1550 2    50   ~ 0
+IRQ_0
 Text Label 2650 1650 2    50   ~ 0
-IRQ_0
-Text Label 2650 1750 2    50   ~ 0
 IRQ_1
-Text Label 2650 1050 2    50   ~ 0
+Text Label 2650 1850 2    50   ~ 0
 NSS_DATA
 Text Label 900  1250 0    50   ~ 0
@@
 SCLK
 Text Label 900  1050 0    50   ~ 0
-IR
-Text Label 900  1750 0    50   ~ 0
+POR
+Text Label 2650 1050 2    50   ~ 0
 STATUS
-Text Label 900  1850 0    50   ~ 0
+Text Label 2650 1450 2    50   ~ 0
 PB_CFG
 Wire Wire Line
@@
 Wire Wire Line
 	2250 1850 2650 1850
-NoConn ~ 2650 1150
+NoConn ~ 900  1850
+NoConn ~ 900  1350
 NoConn ~ 2650 1350
-NoConn ~ 2650 1450
-NoConn ~ 2650 1550
 NoConn ~ 900  1550
 NoConn ~ 900  1650
+NoConn ~ 900  1750
 Wire Notes Line
 	3800 750  3800 2100
 Wire Notes Line
 	750  750  750  2100
-Text Notes 800  4500 0    50   ~ 0
-R: 0805\nC 10u: eletrolitico 4mm (medir)\nSW: 6x6mm smd (duqueeletronica)\nLEDs: 5mm\nBAT: deixar conectores
-$Comp
-L Device:R R8
-U 1 1 5AFCCFBC
-P 5600 2850
-F 0 "R8" H 5670 2896 50  0000 L CNN
-F 1 "0" H 5670 2805 50  0000 L CNN
-F 2 "Resistor_SMD:R_1206_3216Metric_Pad1.24x1.80mm_HandSolder" V 5530 2850 50  0001 C CNN
-F 3 "~" H 5600 2850 50  0001 C CNN
-	1    5600 2850
-	1    0    0    -1
-$EndComp
-Wire Wire Line
-	5600 2600 5600 2700
-Wire Wire Line
-	5600 3000 5600 3100
 Wire Notes Line
 	6000 1950 6000 3200
 Wire Notes Line
 	5050 1950 5050 3200
-$Comp
-L Device:R R4
-U 1 1 5AFD7349
-P 1200 1150
-F 0 "R4" V 1150 1250 50  0000 L CNN
-F 1 "0" V 1200 1150 50  0000 L CNN
-F 2 "Resistor_SMD:R_1206_3216Metric_Pad1.24x1.80mm_HandSolder" V 1130 1150 50  0001 C CNN
-F 3 "~" H 1200 1150 50  0001 C CNN
-	1    1200 1150
-	0    1    1    0
-$EndComp
-$Comp
-L Device:R R5
-U 1 1 5AFDB9E4
-P 1200 1250
-F 0 "R5" V 1150 1350 50  0000 L CNN
-F 1 "0" V 1200 1250 50  0000 L CNN
-F 2 "Resistor_SMD:R_1206_3216Metric_Pad1.24x1.80mm_HandSolder" V 1130 1250 50  0001 C CNN
-F 3 "~" H 1200 1250 50  0001 C CNN
-	1    1200 1250
-	0    1    1    0
-$EndComp
-Wire Wire Line
-	1050 1150 900  1150
-Wire Wire Line
-	1050 1250 900  1250
 Wire Wire Line
 	900  950  1350 950
@@
 Wire Notes Line
 	4950 750  4950 2150
-$Comp
-L Device:R R7
-U 1 1 5AFF7CFB
-P 4500 3900
-F 0 "R7" H 4570 3946 50  0000 L CNN
-F 1 "0" H 4570 3855 50  0000 L CNN
-F 2 "Resistor_SMD:R_1206_3216Metric_Pad1.24x1.80mm_HandSolder" V 4430 3900 50  0001 C CNN
-F 3 "~" H 4500 3900 50  0001 C CNN
-	1    4500 3900
-	1    0    0    -1
-$EndComp
-$Comp
-L Device:R R6
-U 1 1 5B005788
-P 4500 1050
-F 0 "R6" H 4570 1096 50  0000 L CNN
-F 1 "0" H 4570 1005 50  0000 L CNN
-F 2 "Resistor_SMD:R_1206_3216Metric_Pad1.24x1.80mm_HandSolder" V 4430 1050 50  0001 C CNN
-F 3 "~" H 4500 1050 50  0001 C CNN
-	1    4500 1050
-	1    0    0    -1
-$EndComp
+Wire Wire Line
+	4500 3700 4500 4050
+Wire Wire Line
+	5600 2600 5600 3100
+Wire Wire Line
+	4500 850  4500 1200
+Wire Wire Line
+	900  1150 1350 1150
+Wire Wire Line
+	900  1250 1350 1250
 $EndSCHEMATC

Commit message: Replaced Cap Footprint to 5mm
Parts:
- C1: footprint Capacitor_THT:CP_Radial_D4.0mm_P2.00mm -> Capacitor_THT:CP_Radial_D5.0mm_P2.50mm
Changed lines of the file:
@@
 F 0 "C1" H 3250 1300 50  0000 L CNN
 F 1 "10u" H 3250 1100 50  0000 L CNN
-F 2 "Capacitor_THT:CP_Radial_D4.0mm_P2.00mm" H 3238 1050 50  0001 C CNN
+F 2 "Capacitor_THT:CP_Radial_D5.0mm_P2.50mm" H 3238 1050 50  0001 C CNN
 F 3 "~" H 3200 1200 50  0001 C CNN
 	1    3200 1200
